File: DiceRollPcb/DiceRollPcb.sch (KiCad schematic (older format))
At the start: 20 parts, among them SW1 SW_Push, SW2 SW_Push, SW3 SW_Push, SW4 SW_Push, U1 RaspberryPiPico

Commit message: Version 2
Parts:
- added C2: 4.7µF, Capacitor_THT:C_Disc_D4.3mm_W1.9mm_P5.00mm, symbol Device:C
- added D10, D11, D12, D13: D, Diode_THT:D_5W_P12.70mm_Horizontal, symbol Device:D
- added D8, D9: LED, LED_THT:LED_D5.0mm, symbol Device:LED
- added J1: Conn_01x03_Male, Connector_PinHeader_2.54mm:PinHeader_1x03_P2.54mm_Vertical, symbol Connector:Conn_01x03_Male
- added J2: Barrel_Jack, Connector_BarrelJack:BarrelJack_Horizontal, symbol Connector:Barrel_Jack
- added R8, R9: R, Resistor_THT:R_Axial_DIN0207_L6.3mm_D2.5mm_P10.16mm_Horizontal, symbol Device:R
- added SW5, SW6: SW_Push, Button_Switch_THT:SW_PUSH_6mm, symbol Switch:SW_Push
- added U2: R-785.0-0.5, Converter_DCDC:Converter_DCDC_RECOM_R-78E-0.5_THT, symbol Regulator_Switching:R-785.0-0.5
- SW1, SW2, SW3, SW4: footprint Button_Switch_THT:SW_TH_Tactile_Omron_B3F-10xx -> Button_Switch_THT:SW_PUSH_6mm
Connections:
- net +3V3: now also D8.2 (A), D9.2 (A)
- net GND: now also C2.2, D12.2 (A), D13.2 (A), SW5.2, SW6.2, U2.2 (GND)
- net SWITCH1: now also U1.12 (GP9); no longer U1.10 (GP7)
- net SWITCH2: now also U1.14 (GP10); no longer U1.11 (GP8)
- net SWITCH3: now also U1.15 (GP11); no longer U1.12 (GP9)
- net SWITCH4: now also U1.16 (GP12); no longer U1.14 (GP10)
- net SWITCH5: now reaches U1.17 (GP13)
- net SWITCH5: now also SW5.1
- net SWITCH6: now reaches U1.19 (GP14)
- net SWITCH6: now also SW6.1
- net +5V: now reaches U1.40 (VBUS)
- net +5V: now also U2.3 (OUT)
- net at U1.41 (SWCLK): now also J1.1 (Pin_1)
- net at U1.42 (GND): now also J1.2 (Pin_2)
- net at U1.43 (SWDIO): now also J1.3 (Pin_3)
- new net: D8.1 (K), R8.1
- new net: D9.1 (K), R9.1
- new net AC_1: D10.2 (A), D12.1 (K), J2.1
- new net AC_2: D11.2 (A), D13.1 (K), J2.2
- new net DC_PLUS: C2.1, D10.1 (K), D11.1 (K), U2.1 (IN)
- new net LED8: R8.2, U1.10 (GP7)
- new net LED9: R9.2, U1.11 (GP8)
Other:
- moved on the sheet: SW1
